File: kicad documents/HDB-001_Brain_Board/HDB-001_Brain_Board.kicad_pcb (KiCad board)
At the start: 2 copper layers, 75 x 40 mm, 9 parts, among them J1 B2B Sensors/Logic, J2 B2B Commands/Power, J3 SWD/UART/Status placeholder, U1 Black Pill STM32F411CEU6, U2 XIAO ESP32-S3/Plus TBD

Commit message: Advance Rev A0 cockpit firmware and PCB bring-up
Routing:
- net SWDIO: track 0.00 -> 22.7 mm
- net GND: track 0.00 -> 21.9 mm
- net 3V3: track 0.00 -> 21.9 mm
- net SWCLK: track 0.00 -> 21.3 mm
- net NRST: track 0.00 -> 20.9 mm
- net STM32_TX: track 0.00 -> 14.4 mm
- net STM32_RX: track 0.00 -> 14.4 mm
Other:
- board text added: "ESP32-S3-ZERO BENCH: GPIO44<-STM32_TX, GPIO43->STM32_RX, COMMON GND"
- board text added: "J3 DEBUG: SWDIO SWCLK NRST 3V3 GND STM32_TX STM32_RX GND 3V3 GND GND GND"
Changed lines of the file:
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@@
     (effects (font (size 0.8 0.8) (thickness 0.15)) (justify left))
+  )
+  (gr_text "J3 DEBUG: SWDIO SWCLK NRST 3V3 GND STM32_TX STM32_RX GND 3V3 GND GND GND" (at 3 31.8) (layer "F.SilkS")
+    (effects (font (size 0.55 0.55) (thickness 0.08)) (justify left))
+  )
+  (gr_text "ESP32-S3-ZERO BENCH: GPIO44<-STM32_TX, GPIO43->STM32_RX, COMMON GND" (at 3 33.0) (layer "F.SilkS")
+    (effects (font (size 0.55 0.55) (thickness 0.08)) (justify left))
   )
   (footprint "PEGASUS_Placeholders:BlackPill_STM32F411_53x21" (layer "F.Cu")
@@
     (pad "" np_thru_hole circle (at 0 0) (size 2.5 2.5) (drill 2.5) (layers "*.Cu" "*.Mask"))
   )
+  (segment (start 51.810 8.110) (end 37.730 5.000) (width 0.25) (layer "F.Cu") (net 28))
+  (segment (start 54.350 8.110) (end 40.270 5.000) (width 0.25) (layer "F.Cu") (net 27))
+  (segment (start 28.950 25.890) (end 30.110 5.000) (width 0.25) (layer "B.Cu") (net 23))
+  (segment (start 31.490 25.890) (end 27.570 5.000) (width 0.25) (layer "B.Cu") (net 29))
+  (segment (start 34.030 25.890) (end 25.030 5.000) (width 0.25) (layer "B.Cu") (net 30))
+  (segment (start 67.050 8.110) (end 45.350 5.000) (width 0.50) (layer "F.Cu") (net 1))
+  (segment (start 69.590 8.110) (end 47.890 5.000) (width 0.50) (layer "B.Cu") (net 20))
 )
