File: kicad documents/HDB-100_Chassis_Power_Board/HDB-100_Chassis_Power_Board.kicad_pcb (KiCad board)
At the start: 2 copper layers, 182 x 66 mm, 14 parts, among them J1 B2B Sensors/Logic, J2 B2B Commands/Power

Commit message: Advance HDB-100 offline KiCad assembly
Parts:
- added CBULK1: 470-1000uF placeholder, PEGASUS_Placeholders:BulkCap_Radial_D10_P5, F.Cu at (102.0, 27.0)
- added JBAT: XT30 LiPo 2S placeholder, PEGASUS_Placeholders:PowerConnector_1x02_3p5, F.Cu at (174.0, 28.0)
- added J_FAN: Fan/ESC placeholder, PEGASUS_Placeholders:PinHeader_1x04_2p54, F.Cu at (70.0, 58.0)
- added J_ML: Motor L placeholder, PEGASUS_Placeholders:PowerConnector_1x02_3p5, F.Cu at (105.0, 10.0)
- added J_MR: Motor R placeholder, PEGASUS_Placeholders:PowerConnector_1x02_3p5, F.Cu at (150.0, 10.0)
- added SW_PWR: Power switch placeholder, PEGASUS_Placeholders:SlideSwitch_SPST_8x4, F.Cu at (160.0, 10.0)
Other:
- board text added: "ANALOG SENSOR CORRIDOR"
- board text added: "OFFLINE KICAD SPRINT: POWER CONNECTORS ARE PLACEHOLDERS - MEASURE BEFORE GERBER"
- board text added: "Q_FAN OR ESC DRIVER TBD"
- board text added: "VBAT / VMOTOR CORRIDOR"
Changed lines of the file:
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@@
   (net 31 "VBAT_ADC")
   (net 32 "VMOTOR")
+  (net 33 "VBAT_RAW")
   (gr_line (start 0 24) (end 52 24) (stroke (width 0.1) (type solid)) (layer "Edge.Cuts"))
   (gr_line (start 52 24) (end 72 6) (stroke (width 0.1) (type solid)) (layer "Edge.Cuts"))
@@
   (gr_text "High current stays on HDB-100. Keep A0-A7 away from motor/buck/fan." (at 8 69) (layer "Cmts.User")
     (effects (font (size 0.9 0.9) (thickness 0.15)) (justify left))
+  )
+  (gr_text "OFFLINE KICAD SPRINT: POWER CONNECTORS ARE PLACEHOLDERS - MEASURE BEFORE GERBER" (at 8 13) (layer "Cmts.User")
+    (effects (font (size 0.9 0.9) (thickness 0.15)) (justify left))
+  )
+  (gr_text "VBAT / VMOTOR CORRIDOR" (at 141 8.5) (layer "F.SilkS")
+    (effects (font (size 0.9 0.9) (thickness 0.12)))
+  )
+  (gr_text "ANALOG SENSOR CORRIDOR" (at 28 56.5) (layer "F.SilkS")
+    (effects (font (size 0.85 0.85) (thickness 0.12)))
+  )
+  (gr_text "Q_FAN OR ESC DRIVER TBD" (at 75 63.5) (layer "F.SilkS")
+    (effects (font (size 0.75 0.75) (thickness 0.12)))
   )
   (footprint "PEGASUS_Placeholders:Suction_Hole_D22" (layer "F.Cu")
@@
     (pad "12" thru_hole circle (at 13.970 0.000) (size 1.6 1.6) (drill 0.8) (layers "*.Cu" "*.Mask") (net 31 "VBAT_ADC"))
   )
+  (footprint "PEGASUS_Placeholders:PowerConnector_1x02_3p5" (layer "F.Cu")
+    (at 174.000 28.000 0)
+    (property "Reference" "JBAT" (at 0 -3 0) (layer "F.SilkS")
+      (effects (font (size 1 1) (thickness 0.15)))
+    )
+    (property "Value" "XT30 LiPo 2S placeholder" (at 0 3 0) (layer "F.Fab")
+      (effects (font (size 1 1) (thickness 0.15)))
+    )
+    (fp_rect (start -4.8 -2.2) (end 4.8 2.2) (stroke (width 0.12) (type solid)) (fill no) (layer "F.SilkS"))
+    (fp_rect (start -4.8 -2.2) (end 4.8 2.2) (stroke (width 0.1) (type solid)) (fill no) (layer "F.Fab"))
+    (fp_rect (start -5.2 -2.6) (end 5.2 2.6) (stroke (width 0.05) (type solid)) (fill no) (layer "F.CrtYd"))
+    (fp_text user "RAW 2S" (at 0 0 unlocked) (layer "F.SilkS")
+      (effects (font (size 0.7 0.7) (thickness 0.11)))
+    )
+    (pad "1" thru_hole rect (at -1.750 0.000) (size 2.2 2.2) (drill 1.2) (layers "*.Cu" "*.Mask") (net 33 "VBAT_RAW"))
+    (pad "2" thru_hole circle (at 1.750 0.000) (size 2.2 2.2) (drill 1.2) (layers "*.Cu" "*.Mask") (net 20 "GND"))
+  )
+  (footprint "PEGASUS_Placeholders:SlideSwitch_SPST_8x4" (layer "F.Cu")
+    (at 160.000 10.000 0)
+    (property "Reference" "SW_PWR" (at 0 -3.2 0) (layer "F.SilkS")
+      (effects (font (size 1 1) (thickness 0.15)))
+    )
+    (property "Value" "Power switch placeholder" (at 0 3.2 0) (layer "F.Fab")
+      (effects (font (size 1 1) (thickness 0.15)))
+    )
+    (fp_rect (start -4 -2) (end 4 2) (stroke (width 0.12) (type solid)) (fill no) (layer "F.SilkS"))
+    (fp_rect (start -4 -2) (end 4 2) (stroke (width 0.1) (type solid)) (fill no) (layer "F.Fab"))
+    (fp_rect (start -4.4 -2.4) (end 4.4 2.4) (stroke (width 0.05) (type solid)) (fill no) (layer "F.CrtYd"))
+    (fp_text user "ON" (at 2.5 0 unlocked) (layer "F.SilkS")
+      (effects (font (size 0.75 0.75) (thickness 0.12)))
+    )
+    (pad "1" thru_hole rect (at -2.540 0.000) (size 1.8 1.8) (drill 0.9) (layers "*.Cu" "*.Mask") (net 33 "VBAT_RAW"))
+    (pad "2" thru_hole circle (at 2.540 0.000) (size 1.8 1.8) (drill 0.9) (layers "*.Cu" "*.Mask") (net 32 "VMOTOR"))
+  )
+  (footprint "PEGASUS_Placeholders:BulkCap_Radial_D10_P5" (layer "F.Cu")
+    (at 102.000 27.000 0)
+    (property "Reference" "CBULK1" (at 0 -6.4 0) (layer "F.SilkS")
+      (effects (font (size 1 1) (thickness 0.15)))
+    )
+    (property "Value" "470-1000uF placeholder" (at 0 6.4 0) (layer "F.Fab")
+      (effects (font (size 1 1) (thickness 0.15)))
+    )
+    (fp_circle (center 0 0) (end 5 0) (stroke (width 0.12) (type solid)) (fill no) (layer "F.SilkS"))
+    (fp_circle (center 0 0) (end 5 0) (stroke (width 0.1) (type solid)) (fill no) (layer "F.Fab"))
+    (fp_circle (center 0 0) (end 5.4 0) (stroke (width 0.05) (type solid)) (fill no) (layer "F.CrtYd"))
+    (fp_text user "+" (at -3.8 0 unlocked) (layer "F.SilkS")
+      (effects (font (size 1 1) (thickness 0.15)))
+    )
+    (pad "1" thru_hole rect (at -2.500 0.000) (size 1.9 1.9) (drill 0.9) (layers "*.Cu" "*.Mask") (net 32 "VMOTOR"))
+    (pad "2" thru_hole circle (at 2.500 0.000) (size 1.9 1.9) (drill 0.9) (layers "*.Cu" "*.Mask") (net 20 "GND"))
+  )
+  (footprint "PEGASUS_Placeholders:PowerConnector_1x02_3p5" (layer "F.Cu")
+    (at 105.000 10.000 0)
+    (property "Reference" "J_ML" (at 0 -3 0) (layer "F.SilkS")
+      (effects (font (size 1 1) (thickness 0.15)))
+    )
+    (property "Value" "Motor L placeholder" (at 0 3 0) (layer "F.Fab")
+      (effects (font (size 1 1) (thickness 0.15)))
+    )
+    (fp_rect (start -4.8 -2.2) (end 4.8 2.2) (stroke (width 0.12) (type solid)) (fill no) (layer "F.SilkS"))
+    (fp_rect (start -4.8 -2.2) (end 4.8 2.2) (stroke (width 0.1) (type solid)) (fill no) (layer "F.Fab"))
+    (fp_rect (start -5.2 -2.6) (end 5.2 2.6) (stroke (width 0.05) (type solid)) (fill no) (layer "F.CrtYd"))
+    (fp_text user "ML" (at 0 0 unlocked) (layer "F.SilkS")
+      (effects (font (size 0.7 0.7) (thickness 0.11)))
+    )
+    (pad "1" thru_hole rect (at -1.750 0.000) (size 2.2 2.2) (drill 1.2) (layers "*.Cu" "*.Mask") (net 13 "AOUT1"))
+    (pad "2" thru_hole circle (at 1.750 0.000) (size 2.2 2.2) (drill 1.2) (layers "*.Cu" "*.Mask") (net 14 "AOUT2"))
+  )
+  (footprint "PEGASUS_Placeholders:PowerConnector_1x02_3p5" (layer "F.Cu")
+    (at 150.000 10.000 0)
+    (property "Reference" "J_MR" (at 0 -3 0) (layer "F.SilkS")
+      (effects (font (size 1 1) (thickness 0.15)))
+    )
+    (property "Value" "Motor R placeholder" (at 0 3 0) (layer "F.Fab")
+      (effects (font (size 1 1) (thickness 0.15)))
+    )
+    (fp_rect (start -4.8 -2.2) (end 4.8 2.2) (stroke (width 0.12) (type solid)) (fill no) (layer "F.SilkS"))
+    (fp_rect (start -4.8 -2.2) (end 4.8 2.2) (stroke (width 0.1) (type solid)) (fill no) (layer "F.Fab"))
+    (fp_rect (start -5.2 -2.6) (end 5.2 2.6) (stroke (width 0.05) (type solid)) (fill no) (layer "F.CrtYd"))
+    (fp_text user "MR" (at 0 0 unlocked) (layer "F.SilkS")
+      (effects (font (size 0.7 0.7) (thickness 0.11)))
+    )
+    (pad "1" thru_hole rect (at -1.750 0.000) (size 2.2 2.2) (drill 1.2) (layers "*.Cu" "*.Mask") (net 17 "BOUT1"))
+    (pad "2" thru_hole circle (at 1.750 0.000) (size 2.2 2.2) (drill 1.2) (layers "*.Cu" "*.Mask") (net 18 "BOUT2"))
+  )
+  (footprint "PEGASUS_Placeholders:PinHeader_1x04_2p54" (layer "F.Cu")
+    (at 70.000 58.000 0)
+    (property "Reference" "J_FAN" (at 0 -3 0) (layer "F.SilkS")
+      (effects (font (size 1 1) (thickness 0.15)))
+    )
+    (property "Value" "Fan/ESC placeholder" (at 0 3 0) (layer "F.Fab")
+      (effects (font (size 1 1) (thickness 0.15)))
+    )
+    (fp_rect (start -5.35 -1.8) (end 5.35 1.8) (stroke (width 0.12) (type solid)) (fill no) (layer "F.SilkS"))
+    (fp_rect (start -5.65 -2.1) (end 5.65 2.1) (stroke (width 0.05) (type solid)) (fill no) (layer "F.CrtYd"))
+    (pad "1" thru_hole rect (at -3.810 0.000) (size 1.6 1.6) (drill 0.8) (layers "*.Cu" "*.Mask") (net 32 "VMOTOR"))
+    (pad "2" thru_hole circle (at -1.270 0.000) (size 1.6 1.6) (drill 0.8) (layers "*.Cu" "*.Mask") (net 20 "GND"))
+    (pad "3" thru_hole circle (at 1.270 0.000) (size 1.6 1.6) (drill 0.8) (layers "*.Cu" "*.Mask") (net 19 "FAN_PWM"))
+    (pad "4" thru_hole circle (at 3.810 0.000) (size 1.6 1.6) (drill 0.8) (layers "*.Cu" "*.Mask") (net 2 "5V_IN"))
+  )
   (footprint "PEGASUS_Placeholders:MountingHole_2p5_NPTH" (layer "F.Cu")
